Commit message: Pre Mednight

File: f1tenth_gym_ros/launch/ego_racecar.xacro (robot description, xacro)
@@ -2,10 +2,10 @@
 <!-- A simple model of the racecar for rviz -->
 <robot xmlns:xacro="http://www.ros.org/wiki/xacro" name="racecar">
-  <xacro:property name="wheelbase" value="0.3302" />
-  <xacro:property name="width" value="0.2032" />
-  <xacro:property name="height" value="0.1" />
-  <xacro:property name="ground_offset" value="0.04" />
-  <xacro:property name="wheel_radius" value="0.0508" />
-  <xacro:property name="wheel_length" value="0.0381" />
+  <xacro:property name="wheelbase" value="0.3702" />
+  <xacro:property name="width" value="0.294" />
+  <xacro:property name="height" value="0.193" />
+  <xacro:property name="ground_offset" value="0.047" />
+  <xacro:property name="wheel_radius" value="0.11" />
+  <xacro:property name="wheel_length" value="0.069" />
   <xacro:property name="laser_distance_from_base_link" value="0.275" />
   <xacro:property name="laser_height" value="0.05" />
